Commit message: 侧抓改为正上方下压抓取

File: src/orion_description/urdf/orion.urdf (robot description, URDF)
Before this commit: robot orion, 11 links, 10 joints
Links:
- added link gripper_tcp
- link base_link: geometry collision box size=0.6 0.4 0.35; visual mesh filename=../meshes/stl/base_link_left.stl
Joints:
- added joint joint_Link6_gripper_tcp: type fixed, parent Link6, child gripper_tcp, origin xyz=0.0 0.0 0.0499 rpy=0.0 0.0 0.0

File: web/robot/orion.urdf (robot description, URDF)
Before this commit: robot orion, 10 links, 9 joints
Links:
- link base_link: geometry collision mesh filename=meshes/stl/base_link.stl; visual mesh filename=meshes/stl/base_link.stl

Commit message: 优化夹爪抓取位置，工作空间限制

File: src/orion_description/urdf/orion.urdf (robot description, URDF)
Before this commit: robot orion, 12 links, 11 joints
Joints:
- joint joint_Link6_gripper_tcp: origin xyz=0.0 0.0 0.108 rpy=0.0 0.0 0.0 -> xyz=0.0 0.0 0.098 rpy=0.0 0.0 0.0

Commit message: 调整夹爪位置

File: src/orion_description/urdf/orion.urdf (robot description, URDF)
Before this commit: robot orion, 12 links, 11 joints
Joints:
- joint joint_Link6_gripper_tcp: origin xyz=0.0 0.0 0.098 rpy=0.0 0.0 0.0 -> xyz=0.0 0.0 0.128 rpy=0.0 0.0 0.0

Commit message: 调整夹爪抓取的距离

File: src/orion_description/urdf/orion.urdf (robot description, URDF)
Before this commit: robot orion, 12 links, 11 joints
Joints:
- joint joint_Link6_gripper_tcp: origin xyz=0.0 0.0 0.128 rpy=0.0 0.0 0.0 -> xyz=0.0 0.0 0.148 rpy=0.0 0.0 0.0

Commit message: 调整抓取距离，夹爪判定时间优化，窗口+固定时间

File: src/orion_description/urdf/orion.urdf (robot description, URDF)
Before this commit: robot orion, 12 links, 11 joints
Joints:
- joint joint_Link6_gripper_tcp: origin xyz=0.0 0.0 0.148 rpy=0.0 0.0 0.0 -> xyz=0.0 0.0 0.188 rpy=0.0 0.0 0.0

Commit message: 郭工模型更换，把手变成杆

File: src/orion_description/urdf/orion.urdf (robot description, URDF)
Before this commit: robot orion, 12 links, 11 joints
Joints:
- joint joint_Link6_gripper_tcp: origin xyz=0.0 0.0 0.188 rpy=0.0 0.0 0.0 -> xyz=0.0 0.0 0.148 rpy=0.0 0.0 0.0

File: web/robot/orion.urdf (robot description, URDF)
Before this commit: robot orion, 10 links, 9 joints
Links:
- added link gripper_tcp
- added link world
- link base_link: geometry collision box size=0.6 0.4 0.35; visual mesh filename=meshes/stl/base_link_left.stl
Joints:
- added joint joint_Link6_gripper_tcp: type fixed, parent Link6, child gripper_tcp, origin xyz=0.0 0.0 0.148 rpy=0.0 0.0 0.0
- added joint world_joint: type fixed, parent world, child base_link, origin xyz=0.0 0.0 0.0 rpy=0.0 0.0 0.0

Commit message: 添加偏移量，使target对准孔洞，固定抓取位置

File: src/orion_description/urdf/orion.urdf (robot description, URDF)
Before this commit: robot orion, 12 links, 11 joints
Links:
- added link peg_tip
Joints:
- added joint joint_gripper_tcp_peg_tip: type fixed, parent gripper_tcp, child peg_tip, origin xyz=0.0 0.08 0.035 rpy=0.0 0.0 0.0

File: web/robot/orion.urdf (robot description, URDF)
Before this commit: robot orion, 12 links, 11 joints
Links:
- added link peg_tip
Joints:
- added joint joint_gripper_tcp_peg_tip: type fixed, parent gripper_tcp, child peg_tip, origin xyz=0.0 0.08 0.035 rpy=0.0 0.0 0.0

Commit message: 引入trakIK，增加大角度限制，优先小角度抓取。急停停止所有任务

File: src/orion_description/urdf/orion.urdf (robot description, URDF)
Before this commit: robot orion, 13 links, 12 joints
Joints:
- joint joint_Link5_Link6: limit effort=100 velocity=1.0 -> lower=-3.14159 upper=3.14159 effort=100 velocity=1.0; type continuous -> revolute

File: web/robot/orion.urdf (robot description, URDF)
Before this commit: robot orion, 13 links, 12 joints
Joints:
- joint joint_Link5_Link6: limit effort=100 velocity=1.0 -> lower=-3.14159 upper=3.14159 effort=100 velocity=1.0; type continuous -> revolute

Commit message: 解决插孔方向相反问题，增加插入锁存时撤回重规划

File: src/orion_description/urdf/orion.urdf (robot description, URDF)
Before this commit: robot orion, 13 links, 12 joints
Joints:
- joint joint_gripper_tcp_peg_tip: origin xyz=0.0 0.08 0.035 rpy=0.0 0.0 0.0 -> xyz=0.0 -0.08 0.035 rpy=0.0 0.0 0.0

File: web/robot/orion.urdf (robot description, URDF)
Before this commit: robot orion, 13 links, 12 joints
Joints:
- joint joint_gripper_tcp_peg_tip: origin xyz=0.0 0.08 0.035 rpy=0.0 0.0 0.0 -> xyz=0.0 -0.08 0.035 rpy=0.0 0.0 0.0
