Commit message: 1、增加关节限位

File: rov_urdf/orion_left.urdf (robot description, URDF)
Before this commit: robot orion, 10 links, 9 joints
Joints:
- joint joint_Link1_Link2: limit lower=-3.14159 upper=3.14159 effort=100 velocity=1.0 -> lower=-2.09440 upper=2.09440 effort=100 velocity=1.0
- joint joint_Link2_Link3: limit lower=-3.14159 upper=3.14159 effort=100 velocity=1.0 -> lower=-2.09440 upper=2.09440 effort=100 velocity=1.0
- joint joint_Link4_Link5: limit lower=-3.14159 upper=3.14159 effort=100 velocity=1.0 -> lower=-2.09440 upper=2.09440 effort=100 velocity=1.0
- joint joint_Link5_Link6: limit lower=-3.14159 upper=3.14159 effort=100 velocity=1.0 -> effort=100 velocity=1.0; type revolute -> continuous
- joint joint_LinkVirtual_Link4: limit lower=-3.14159 upper=3.14159 effort=100 velocity=1.0 -> lower=-4.71239 upper=4.71239 effort=100 velocity=1.0
- joint joint_base_link_Link1: limit lower=-3.14159 upper=3.14159 effort=100 velocity=1.0 -> lower=-2.09440 upper=2.09440 effort=100 velocity=1.0

File: rov_urdf/orion_right.urdf (robot description, URDF)
Before this commit: robot orion, 10 links, 9 joints
Joints:
- joint joint_Link1_Link2: limit lower=-3.14159 upper=3.14159 effort=100 velocity=1.0 -> lower=-2.09440 upper=2.09440 effort=100 velocity=1.0
- joint joint_Link2_Link3: limit lower=-3.14159 upper=3.14159 effort=100 velocity=1.0 -> lower=-2.09440 upper=2.09440 effort=100 velocity=1.0
- joint joint_Link4_Link5: limit lower=-3.14159 upper=3.14159 effort=100 velocity=1.0 -> lower=-2.09440 upper=2.09440 effort=100 velocity=1.0
- joint joint_Link5_Link6: limit lower=-3.14159 upper=3.14159 effort=100 velocity=1.0 -> effort=100 velocity=1.0; type revolute -> continuous
- joint joint_LinkVirtual_Link4: limit lower=-3.14159 upper=3.14159 effort=100 velocity=1.0 -> lower=-4.71239 upper=4.71239 effort=100 velocity=1.0
- joint joint_base_link_Link1: limit lower=-3.14159 upper=3.14159 effort=100 velocity=1.0 -> lower=-2.09440 upper=2.09440 effort=100 velocity=1.0

File: src/orion_description/urdf/orion.urdf (robot description, URDF)
Before this commit: robot orion, 12 links, 11 joints
Joints:
- joint joint_Link1_Link2: limit lower=-3.14159 upper=3.14159 effort=100 velocity=1.0 -> lower=-2.09440 upper=2.09440 effort=100 velocity=1.0
- joint joint_Link2_Link3: limit lower=-3.14159 upper=3.14159 effort=100 velocity=1.0 -> lower=-2.09440 upper=2.09440 effort=100 velocity=1.0
- joint joint_Link4_Link5: limit lower=-3.14159 upper=3.14159 effort=100 velocity=1.0 -> lower=-2.09440 upper=2.09440 effort=100 velocity=1.0
- joint joint_Link5_Link6: limit lower=-3.14159 upper=3.14159 effort=100 velocity=1.0 -> effort=100 velocity=1.0; type revolute -> continuous
- joint joint_LinkVirtual_Link4: limit lower=-3.14159 upper=3.14159 effort=100 velocity=1.0 -> lower=-4.71239 upper=4.71239 effort=100 velocity=1.0
- joint joint_base_link_Link1: limit lower=-3.14159 upper=3.14159 effort=100 velocity=1.0 -> lower=-2.09440 upper=2.09440 effort=100 velocity=1.0

File: web/robot/orion.urdf (robot description, URDF)
Before this commit: robot orion, 10 links, 9 joints
Joints:
- joint joint_Link1_Link2: limit lower=-3.14159 upper=3.14159 effort=100 velocity=1.0 -> lower=-2.09440 upper=2.09440 effort=100 velocity=1.0
- joint joint_Link2_Link3: limit lower=-3.14159 upper=3.14159 effort=100 velocity=1.0 -> lower=-2.09440 upper=2.09440 effort=100 velocity=1.0
- joint joint_Link4_Link5: limit lower=-3.14159 upper=3.14159 effort=100 velocity=1.0 -> lower=-2.09440 upper=2.09440 effort=100 velocity=1.0
- joint joint_Link5_Link6: limit lower=-3.14159 upper=3.14159 effort=100 velocity=1.0 -> effort=100 velocity=1.0; type revolute -> continuous
- joint joint_LinkVirtual_Link4: limit lower=-3.14159 upper=3.14159 effort=100 velocity=1.0 -> lower=-4.71239 upper=4.71239 effort=100 velocity=1.0
- joint joint_base_link_Link1: limit lower=-3.14159 upper=3.14159 effort=100 velocity=1.0 -> lower=-2.09440 upper=2.09440 effort=100 velocity=1.0

Commit message: joint4从270改成180

File: rov_urdf/orion_left.urdf (robot description, URDF)
Before this commit: robot orion, 10 links, 9 joints
Joints:
- joint joint_LinkVirtual_Link4: limit lower=-4.71239 upper=4.71239 effort=100 velocity=1.0 -> lower=-3.14159 upper=3.14159 effort=100 velocity=1.0

File: rov_urdf/orion_right.urdf (robot description, URDF)
Before this commit: robot orion, 10 links, 9 joints
Joints:
- joint joint_LinkVirtual_Link4: limit lower=-4.71239 upper=4.71239 effort=100 velocity=1.0 -> lower=-3.14159 upper=3.14159 effort=100 velocity=1.0

File: src/orion_description/urdf/orion.urdf (robot description, URDF)
Before this commit: robot orion, 12 links, 11 joints
Joints:
- joint joint_LinkVirtual_Link4: limit lower=-4.71239 upper=4.71239 effort=100 velocity=1.0 -> lower=-3.14159 upper=3.14159 effort=100 velocity=1.0

File: web/robot/orion.urdf (robot description, URDF)
Before this commit: robot orion, 10 links, 9 joints
Joints:
- joint joint_LinkVirtual_Link4: limit lower=-4.71239 upper=4.71239 effort=100 velocity=1.0 -> lower=-3.14159 upper=3.14159 effort=100 velocity=1.0

Commit message: 手柄和夹爪同步限制空间，夹爪都设为90度

File: rov_urdf/orion_left.urdf (robot description, URDF)
Before this commit: robot orion, 10 links, 9 joints
Joints:
- joint joint_Link6_Link7: limit lower=-3.14159 upper=3.14159 effort=100 velocity=1.0 -> lower=-1.57080 upper=1.57080 effort=100 velocity=1.0
- joint joint_Link6_Link8: limit lower=-3.14159 upper=3.14159 effort=100 velocity=1.0 -> lower=-1.57080 upper=1.57080 effort=100 velocity=1.0

File: rov_urdf/orion_right.urdf (robot description, URDF)
Before this commit: robot orion, 10 links, 9 joints
Joints:
- joint joint_Link6_Link7: limit lower=-3.14159 upper=3.14159 effort=100 velocity=1.0 -> lower=-1.57080 upper=1.57080 effort=100 velocity=1.0
- joint joint_Link6_Link8: limit lower=-3.14159 upper=3.14159 effort=100 velocity=1.0 -> lower=-1.57080 upper=1.57080 effort=100 velocity=1.0

File: src/orion_description/urdf/orion.urdf (robot description, URDF)
Before this commit: robot orion, 12 links, 11 joints
Joints:
- joint joint_Link6_Link7: limit lower=-3.14159 upper=3.14159 effort=100 velocity=1.0 -> lower=-1.57080 upper=1.57080 effort=100 velocity=1.0
- joint joint_Link6_Link8: limit lower=-3.14159 upper=3.14159 effort=100 velocity=1.0 -> lower=-1.57080 upper=1.57080 effort=100 velocity=1.0

File: web/robot/orion.urdf (robot description, URDF)
Before this commit: robot orion, 10 links, 9 joints
Joints:
- joint joint_Link6_Link7: limit lower=-3.14159 upper=3.14159 effort=100 velocity=1.0 -> lower=-1.57080 upper=1.57080 effort=100 velocity=1.0
- joint joint_Link6_Link8: limit lower=-3.14159 upper=3.14159 effort=100 velocity=1.0 -> lower=-1.57080 upper=1.57080 effort=100 velocity=1.0

Commit message: 1、联调东东视觉+陆工任务转发成功。2、修改项目TF链接的baselink名字。3、前端根据郭工armsensor的值实时更新，不桥接。

File: rov_urdf/orion_left.urdf (robot description, URDF)
Before this commit: robot orion, 10 links, 9 joints
Links:
- removed link base_link
- added link arm_base_link, mass 1.0; visual mesh filename=meshes/stl/arm_base_link_left.stl
Joints:
- removed joint joint_base_link_Link1
- added joint joint_arm_base_link_Link1: type revolute, parent arm_base_link, child Link1, origin xyz=0.0 0.0 0.0 rpy=0.0 0.0 0.0, axis 1 0 0, limit lower=-2.09440 upper=2.09440 effort=100 velocity=1.0

File: rov_urdf/orion_right.urdf (robot description, URDF)
Before this commit: robot orion, 10 links, 9 joints
Links:
- removed link base_link
- added link arm_base_link, mass 1.0; visual mesh filename=meshes/stl/arm_base_link_right.stl
Joints:
- removed joint joint_base_link_Link1
- added joint joint_arm_base_link_Link1: type revolute, parent arm_base_link, child Link1, origin xyz=0.0 0.0 0.0 rpy=0.0 0.0 0.0, axis 1 0 0, limit lower=-2.09440 upper=2.09440 effort=100 velocity=1.0

File: src/orion_description/urdf/orion.urdf (robot description, URDF)
Before this commit: robot orion, 13 links, 12 joints
Links:
- removed link base_link
- added link arm_base_link, mass 1.0; collision box size=0.6 0.4 0.35; visual mesh filename=../meshes/stl/arm_base_link_left.stl
Joints:
- removed joint joint_base_link_Link1
- added joint joint_arm_base_link_Link1: type revolute, parent arm_base_link, child Link1, origin xyz=0.0 0.0 0.0 rpy=0.0 0.0 0.0, axis 1 0 0, limit lower=-2.09440 upper=2.09440 effort=100 velocity=1.0
- joint world_joint: child base_link -> arm_base_link

File: web/robot/orion.urdf (robot description, URDF)
Before this commit: robot orion, 13 links, 12 joints
Links:
- removed link base_link
- added link arm_base_link, mass 1.0; collision box size=0.6 0.4 0.35; visual mesh filename=meshes/stl/arm_base_link_left.stl
Joints:
- removed joint joint_base_link_Link1
- added joint joint_arm_base_link_Link1: type revolute, parent arm_base_link, child Link1, origin xyz=0.0 0.0 0.0 rpy=0.0 0.0 0.0, axis 1 0 0, limit lower=-2.09440 upper=2.09440 effort=100 velocity=1.0
- joint world_joint: child base_link -> arm_base_link
